File: SAFE LOCKOUT.kicad_pcb (KiCad board)
At the start: 2 copper layers, 42 parts, among them J1 Conn_01x08_Pin, J10 Conn_01x02_Pin, J2 Conn_01x02_Pin, J3 Conn_01x02_Pin, J4 Conn_01x02_Pin, J5 Conn_01x02_Pin, J6 Conn_01x02_Pin, J7 Conn_01x02_Pin, J8 Conn_01x02_Pin, J9 Conn_01x02_Pin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

Commit message: logan did pcb, some suff still needs to be fixed
Parts:
- D1, D2, D3, D4, D5, D6, D7: footprint digikey-footprints:DO-214AC -> Solenoid Safeguard:DO-214AC
- J1: value Conn_01x08_Pin -> Conn_01x12_Pin; footprint Connector_Molex:Molex_Micro-Fit_3.0_43045-1600_2x08_P3.00mm_Horizontal -> 430451200:MOLEX_430451200
- J2: footprint Connector_JST:JST_XH_B2B-XH-AM_1x02_P2.50mm_Vertical -> Connector_Molex:Molex_Micro-Fit_3.0_43650-0200_1x02_P3.00mm_Horizontal
- J9: footprint Connector_Phoenix_MSTB:PhoenixContact_MSTBVA_2,5_2-G_1x02_P5.00mm_Vertical -> Kinky:PhoenixContact_MSTBVA_2,5_2-G_1x02_P5.00mm_Vertical
- K1: footprint PR30_24V_450_1A:RELAY_PR30-24V-450-1A -> Solenoid Safeguard:RELAY_PR30-24V-450-1A
- Q1, Q2, Q3, Q4, Q5, Q6, Q7, Q8: footprint digikey-footprints:SOT-23-3 -> Package_TO_SOT_SMD:SOT-23-3
- R1, R11, R13, R15, R3, R5, R7, R9: footprint PCM_JLCPCB:R_0805 -> Solenoid Safeguard:R_0805
- R10, R12, R14, R16, R2, R4, R6, R8: footprint Resistor_SMD:R_0402_1005Metric -> Solenoid Safeguard:R_0805
- moved J1 137.4 mm to (70.0, 169.2)
- moved J3 126.9 mm to (48.0, 152.8), turned to -90 degrees
- moved D1 125.1 mm to (54.8, 154.0), turned to -90 degrees
- moved R1 124.8 mm to (63.8, 160.0), turned to 90 degrees
- moved R2 124.5 mm to (63.8, 156.0), turned to -90 degrees
- moved Q1 117.8 mm to (59.4, 156.0), turned to 180 degrees
- moved R4 116.8 mm to (63.8, 146.0), turned to -90 degrees
- moved R3 115.9 mm to (63.5, 151.2), turned to 90 degrees
- moved D2 113.6 mm to (54.8, 144.0), turned to -90 degrees
- moved Q2 113.3 mm to (59.2, 146.0), turned to 180 degrees
- moved J4 112.2 mm to (48.0, 142.8), turned to -90 degrees
- moved R6 109.7 mm to (63.8, 135.8), turned to -90 degrees
- moved J9 109.0 mm to (93.5, 161.2), turned to 90 degrees
- moved R5 105.7 mm to (63.8, 140.2), turned to 90 degrees
- moved J10 104.6 mm to (88.2, 168.5), turned to 180 degrees
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Connections:
- J1 pad 1: VLV 1 CTL -> GND
- J1 pad 10: (no net) -> VLV 3 CTL
- J1 pad 11: (no net) -> VLV 2 CTL
- J1 pad 12: (no net) -> VLV 1 CTL
- J1 pad 2: VLV 2 CTL -> IGNITOR CTL
- J1 pad 3: VLV 3 CTL -> RELAY SFEGRD CTL
- J1 pad 4: VLV 4 CTL -> unconnected-(J1-Pin_4-Pad4)
- J1 pad 5: AV FILL CTL -> unconnected-(J1-Pin_5-Pad5)
- J1 pad 6: AV  RUN CTL -> unconnected-(J1-Pin_6-Pad6)
- J1 pad 7: IGNITOR CTL -> AV FILL CTL
- J1 pad 8: RELAY SFEGRD CTL -> AV  RUN CTL
- J1 pad 9: (no net) -> VLV 4 CTL
Routing:
- net +24V: track 0.00 -> 166.1 mm
- net SAFE POWER 24v: track 0.00 -> 118.5 mm
- net AV FILL CTL: track 0.00 -> 59.7 mm
- net AV  RUN CTL: track 0.00 -> 51.4 mm
- net VLV 4 CTL: track 0.00 -> 39.5 mm
- net IGNITOR CTL: track 0.00 -> 38.5 mm, vias 0 -> 3
- net RELAY SFEGRD CTL: track 0.00 -> 36.4 mm, vias 0 -> 2
- net VLV 3 CTL: track 0.00 -> 31.4 mm
- net Net-(Q8-D): track 0.00 -> 26.2 mm, vias 0 -> 1
- net GND: track 0.00 -> 24.1 mm
- net Net-(J9-Pin_2): track 0.00 -> 21.3 mm
- net VLV 2 CTL: track 0.00 -> 21.1 mm
- net IGNITOR 3A -: track 0.00 -> 17.5 mm
- net Net-(Q7-G): track 0.00 -> 13.3 mm, vias 0 -> 2
- net AV FILL VLV: track 0.00 -> 11.2 mm
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Other:
- board outline added: 68.8 x 88.2 mm
